Commit message: fully switch to urdf

File: dimos/robot/unitree/go2/go2.urdf (robot description, URDF)
Before this commit: robot go2, 1 links, 0 joints
Links:
- added link camera_link
- added link camera_optical
Joints:
- added joint base_link_to_camera_link: type fixed, parent base_link, child camera_link, origin xyz=0.3 0.0 0.0 rpy=0 0 0
- added joint camera_link_to_camera_optical: type fixed, parent camera_link, child camera_optical, origin xyz=0.0 0.0 0.0 rpy=-1.5707963267948966 0 -1.5707963267948966
