Commit message: go2 reframer

File: dimos/mapping/recording/go2_mid360/static_transforms.urdf (robot description, URDF)
Before this commit: robot go2, 5 links, 4 joints
Links:
- added link imu_frame
- added link lidar_frame
- link mid360_link: geometry visual box size=0.065 0.065 0.06
Joints:
- added joint lidar_frame_to_imu_frame: type fixed, parent lidar_frame, child imu_frame, origin xyz=0.011 0.02329 -0.04412 rpy=0 0 0
- added joint mid360_link_to_lidar_frame: type fixed, parent mid360_link, child lidar_frame, origin xyz=0 0 0.017 rpy=0 0 0
