Commit message: render time

File: dimos/robot/unitree/go2/blueprints/navigation/go2_mid360_normal.urdf (robot description, URDF)
Before this commit: robot go2_mid360, 4 links, 3 joints
Joints:
- joint front_camera_to_mid360_link: origin xyz=-0.032 0.0 0.12 rpy=0.0 0.767944870877505 0.0 -> xyz=-0.032 0.0 0.12 rpy=0.0 0.0 0.0
