Commit message: fix(g1): mid360_joint carries the real upside-down mount (roll pi)
The MID-360 is physically mounted inverted on the G1 head; the URDF
had only the 2.3 deg pitch. Measured live: FAST-LIO odometry reports
the sensor body rolled ~180 deg relative to its gravity-aligned world
frame while the robot stands upright, and the pimsim lidar calibration
already used roll=180. With the corrected joint, composing odometry
with the model's inverse pelvis->mid360 transform yields a pelvis
within 1.4 deg of upright (was: robot mesh rendered upside down).

File: dimos/robot/unitree/g1/g1.urdf (robot description, URDF)
Before this commit: robot g1_29dof_rev_1_0, 40 links, 39 joints
Joints:
- joint mid360_joint: origin xyz=0.0002835 0.00003 0.41618 rpy=0 0.04014257279586953 0 -> xyz=0.0002835 0.00003 0.41618 rpy=3.141592653589793 0.04014257279586953 0
