Commit message: organize, untested

File: dimos/robot/bosdyn/spot/spot.urdf (robot description, URDF)
Before this commit: robot spot, 19 links, 18 joints
Links:
- added link back_camera
- added link back_camera_optical
- added link frontleft_camera
- added link frontleft_camera_optical
- added link frontright_camera
- added link frontright_camera_optical
- added link left_camera
- added link left_camera_optical
- added link right_camera
- added link right_camera_optical
Joints:
- added joint back_camera_joint: type fixed, parent body, child back_camera, origin xyz=-0.425 0 0.01 rpy=0 0.3 -3.1415927
- added joint back_camera_optical_joint: type fixed, parent back_camera, child back_camera_optical, origin xyz=0 0 0 rpy=-1.5707963 0 -1.5707963
- added joint frontleft_camera_joint: type fixed, parent body, child frontleft_camera, origin xyz=0.415 0.037 -0.01 rpy=1.355558 0.353917 -0.554196
- added joint frontleft_camera_optical_joint: type fixed, parent frontleft_camera, child frontleft_camera_optical, origin xyz=0 0 0 rpy=-1.5707963 0 -1.5707963
- added joint frontright_camera_joint: type fixed, parent body, child frontright_camera, origin xyz=0.415 -0.037 -0.01 rpy=-1.355558 0.353917 0.554196
- added joint frontright_camera_optical_joint: type fixed, parent frontright_camera, child frontright_camera_optical, origin xyz=0 0 0 rpy=-1.5707963 0 -1.5707963
- added joint left_camera_joint: type fixed, parent body, child left_camera, origin xyz=-0.125 0.12 0.035 rpy=0 0.2 1.5707963
- added joint left_camera_optical_joint: type fixed, parent left_camera, child left_camera_optical, origin xyz=0 0 0 rpy=-1.5707963 0 -1.5707963
- added joint right_camera_joint: type fixed, parent body, child right_camera, origin xyz=-0.125 -0.12 0.035 rpy=0 0.2 -1.5707963
- added joint right_camera_optical_joint: type fixed, parent right_camera, child right_camera_optical, origin xyz=0 0 0 rpy=-1.5707963 0 -1.5707963
