Commit message: fix: drive stereo_mount recording with Point-LIO so world resolves
- Swap raw Mid360 for PointLio(frame_id=world, sensor_frame_id=lidar_link):
  odometry publishes the moving world->lidar_link edge onto tf
- Rename urdf frame lidar_frame->lidar_link so the odometry edge ties into
  the rig tree (frame names must match exactly for tf lookups)
- StereoMountRecorder now extends PointlioRecorder (odometry-baked poses)

Live-tested: all streams world-anchored (249/254 images with poses), zero
'No direct transform' warnings.

File: dimos/robot/assembly/stereo_mount/stereo_mount.urdf (robot description, URDF)
Before this commit: robot stereo_mount, 9 links, 8 joints
Links:
- removed link lidar_frame
- added link lidar_link
Joints:
- joint mid360_to_lidar: child lidar_frame -> lidar_link
